File: PCB/IR-sensor-A2/IR-sensor.kicad_pcb (KiCad board)
At the start: 4 copper layers, 90 x 20 mm, 58 parts, among them J2 Conn_02x10_Odd_Even, J3 Conn_02x10_Odd_Even, Q1 BSS138, Q2 BSS138, U1 MCP6004, U2 HX6206P252MR, U4 TPS60400DBVR

Commit message: Rev A2 received, board bring-up on A2
Routing:
- net /DOG_5: track 128.7 -> 130.4 mm
- net /PWM_SEND: track 144.2 -> 142.6 mm
- net +5V: track 10.7 -> 11.7 mm
- net /DOG_6: track 117.6 -> 118.2 mm
- net /DOG_4: track 139.4 -> 138.8 mm, vias 5 -> 4
- net GND: vias 36 -> 18
