File: PCB/IR-sensor-A2/IR-sensor.kicad_sch (KiCad schematic)
At the start: 58 parts, among them J2 Conn_02x10_Odd_Even, J3 Conn_02x10_Odd_Even, Q1 BSS138, Q2 BSS138, U1 MCP6004, U2 HX6206P252MR, U4 TPS60400DBVR

Commit message: Rev A2 received, board bring-up on A2
Parts:
- D5, D6, JP1, JP10, JP11, JP12, JP13, JP14, JP2, JP3, JP4, JP5, JP6, JP7, JP8, JP9: now left out of the parts list
- R11: MPN RC0402FR-07200RL -> 0402WGF2000TCE; SPN C114764 -> C25087
- R14, R16, R3, R5: MPN RC0402FR-071KL -> 0402WGF1001TCE; SPN C2935237 -> C11702
Other:
- moved on the sheet: C11, C13, R16, R17, R18, U1D
