File: PCB/Receiver-A2/Receiver.kicad_pcb (KiCad board)
At the start: 4 copper layers, 101 x 25.5 mm, 33 parts, among them J10 Conn_02x10_Odd_Even, J6 USB_C_Receptacle_USB2.0, J8 Conn_01x04_Pin, SW1 SW_Push, SW2 SW_Push, U1 TD8102, U2 ESP32-S3-WROOM-1, Y1 Crystal

Commit message: Rev A2 received, board bring-up on A2
Parts:
- U2: footprint PCM_Espressif:ESP32-S3-WROOM-1 -> Devent:ESP32-S3-WROOM-1
- moved C5 0.38 mm to (147.9, 50.4)
Routing:
- net +5V: track 83.9 -> 98.6 mm, vias 4 -> 0
