File: PCB/Receiver-A2/Receiver.kicad_sch (KiCad schematic)
At the start: 33 parts, among them J10 Conn_02x10_Odd_Even, J35 USB_C_Receptacle_USB2.0, J8 Conn_01x04_Pin, SW1 SW_Push, SW2 SW_Push, U1 TD8102, U2 ESP32-S3-WROOM-1, Y1 Crystal

Commit message: Rev A2 received, board bring-up on A2
Parts:
- SW1, SW2: SPN C354948 -> C557592
- U2: footprint PCM_Espressif:ESP32-S3-WROOM-1 -> Devent:ESP32-S3-WROOM-1
Connections:
- no-connect marks 9 -> 15
